File: design/nano_signals.kicad_pcb (KiCad board)
At the start: 2 copper layers, 56.1 x 67.7 mm, 46 parts, among them J1 Conn_01x02_Pin, J2 DCC, J3 Conn_01x02_Pin, J5 D11 D10 D9 D8 D7 D6 D5 D4 D3 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, J6 D12 D13 A0 A1 A2 A3 A4 A5 A6 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, SW1 Prgm A7, U1 6N137, U2 L7805

Commit message: v2 & production
Parts:
- added REF**: MountingHole_2.2mm_M2, MountingHole:MountingHole_2.2mm_M2, F.Cu at (112.4, 88.9)
- added REF**: MountingHole_2.2mm_M2, MountingHole:MountingHole_2.2mm_M2, F.Cu at (104.8, 149.5)
- added REF**: MountingHole_2.2mm_M2, MountingHole:MountingHole_2.2mm_M2, F.Cu at (129.0, 149.5)
- moved D3 1.83 mm to (111.9, 94.4)
- moved D2 1.40 mm to (124.7, 92.1)
- moved J1 0.33 mm to (106.4, 90.8)
Routing:
- net GNDD: track 123.7 -> 119.5 mm
- net Net-(J3-Pin_1): track 8.86 -> 12.0 mm
- net Net-(J1-Pin_1): track 9.59 -> 11.2 mm
- net Net-(D3-A): track 5.39 -> 4.34 mm
- net Net-(D2-+): track 18.3 -> 17.7 mm
