File: design/nano_signals.kicad_sch (KiCad schematic)
At the start: 46 parts, among them J1 Conn_01x02_Pin, J2 DCC, J3 Conn_01x02_Pin, J5 D11 D10 D9 D8 D7 D6 D5 D4 D3 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, J6 D12 D13 A0 A1 A2 A3 A4 A5 A6 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, SW1 Prgm A7, U1 6N137, U2 L7805

Commit message: v2 & production
Parts:
- added J4: DCC, TerminalBlock_4Ucon:TerminalBlock_4Ucon_1x02_P3.50mm_Horizontal, symbol Connector:Screw_Terminal_01x02
Connections:
- net at D2.3, J3.1 (Pin_1): now also J4.2 (Pin_2)
- net at D2.4, J1.1 (Pin_1): now also J4.1 (Pin_1)
Other:
- title: (none) -> MrJ-Train-Signals-DCC-PCB
Changed lines of the file:
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@@
 (kicad_sch (version 20230121) (generator eeschema)
   (paper "A4")
+  (title_block
+    (title "MrJ-Train-Signals-DCC-PCB")
+    (date "2024-11-15")
+    (rev "v2.0")
+    (comment 1 "Custom PCB designed to work with")
+    (comment 2 "https://github.com/HO44-PROJECT/MrJ-HO-scale-DB-style-Era-III-Train-Signals-Electronics")
+    (comment 3 "This PCB needs a Nano to drive my Train Signals")
+  )
   (junction (at 180.34 40.64) (diameter 0) (color 0 0 0 0)
   )
@@
   (junction (at 176.53 83.82) (diameter 0) (color 0 0 0 0)
   )
+  (junction (at 73.66 19.05) (diameter 0) (color 0 0 0 0)
+  )
   (junction (at 48.26 48.26) (diameter 0) (color 0 0 0 0)
   )
@@
   (junction (at 217.17 40.64) (diameter 0) (color 0 0 0 0)
   )
+  (junction (at 74.93 13.97) (diameter 0) (color 0 0 0 0)
+  )
   (junction (at 68.58 40.64) (diameter 0) (color 0 0 0 0)
   )
@@
     (stroke (width 0) (type default))
   )
+  (wire (pts (xy 74.93 13.97) (xy 74.93 26.67))
+    (stroke (width 0) (type default))
+  )
   (wire (pts (xy 62.23 40.64) (xy 63.5 40.64))
     (stroke (width 0) (type default))
@@
     (stroke (width 0) (type default))
   )
+  (wire (pts (xy 74.93 13.97) (xy 135.89 13.97))
+    (stroke (width 0) (type default))
+  )
   (wire (pts (xy 228.6 25.4) (xy 231.14 25.4))
     (stroke (width 0) (type default))
@@
     (stroke (width 0) (type default))
   )
+  (wire (pts (xy 74.93 29.21) (xy 73.66 29.21))
+    (stroke (width 0) (type default))
+  )
   (wire (pts (xy 137.16 113.03) (xy 138.43 113.03))
     (stroke (width 0) (type default))
@@
     (stroke (width 0) (type default))
   )
+  (wire (pts (xy 73.66 19.05) (xy 157.48 19.05))
+    (stroke (width 0) (type default))
+  )
   (wire (pts (xy 217.17 25.4) (xy 213.36 25.4))
     (stroke (width 0) (type default))
@@
     (stroke (width 0) (type default))
   )
-  (wire (pts (xy 52.07 19.05) (xy 157.48 19.05))
+  (wire (pts (xy 52.07 19.05) (xy 73.66 19.05))
     (stroke (width 0) (type default))
   )
@@
     (stroke (width 0) (type default))
   )
+  (wire (pts (xy 73.66 19.05) (xy 73.66 29.21))
+    (stroke (width 0) (type default))
+  )
   (wire (pts (xy 114.3 73.66) (xy 114.3 76.2))
     (stroke (width 0) (type default))
@@
     (stroke (width 0) (type default))
   )
-  (wire (pts (xy 39.37 13.97) (xy 135.89 13.97))
+  (wire (pts (xy 39.37 13.97) (xy 74.93 13.97))
     (stroke (width 0) (type default))
   )
@@
         )
       )
+    )
+  )
+  (symbol (lib_id "Connector:Screw_Terminal_01x02") (at 80.01 29.21 0) (mirror x) (unit 1)
+    (in_bom yes) (on_board yes) (dnp no)
+    (property "Reference" "J4" (at 80.01 20.32 0)
+      (effects (font (size 1.27 1.27)))
+    )
+    (property "Value" "DCC" (at 80.01 22.86 0)
+      (effects (font (size 1.27 1.27)) hide)
+    )
+    (property "Footprint" "TerminalBlock_4Ucon:TerminalBlock_4Ucon_1x02_P3.50mm_Horizontal" (at 80.01 29.21 0)
+      (effects (font (size 1.27 1.27)) hide)
+    )
+    (property "Datasheet" "~" (at 80.01 29.21 0)
+      (effects (font (size 1.27 1.27)) hide)
+    )
+    (pin "1")
+    (pin "2")
+    (instances
+      (project "nano_signals"
+        (path "/a0ad67ff-9d84-4687-83ea-0beba130a41e"
+          (reference "J4") (unit 1)
+        )
+      )
